File: hw/blemesh.kicad_pcb (KiCad board)
At the start: 2 copper layers, 35.6 x 22.9 mm, 73 parts, among them J1 Conn_01x04, J2 CONN_1X03, J3 CONN_1X03, J4 Conn_01x06, J5 TC2030-CTX, U1 NRF52810-QCAA, U2 MIC550X, Y1 32Mhz

Commit message: Removed paste layer from tag connect footprint
Parts:
- J5: footprint alvarop:TC2030-NL -> TC2030-NL
Changed lines of the file:
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@@
-(kicad_pcb (version 4) (host pcbnew 4.0.7-e2-6376~58~ubuntu16.04.1)
+(kicad_pcb (version 4) (host pcbnew 4.0.7+dfsg1-1ubuntu2)
   (general
     (links 117)
@@
     (33 F.Adhes user)
     (34 B.Paste user)
-    (35 F.Paste user)
+    (35 F.Paste user hide)
     (36 B.SilkS user)
     (37 F.SilkS user)
@@
     (add_net "Net-(U2-Pad4)")
   )
+  (module TC2030-NL (layer F.Cu)
+    (at 187.198 99.441)
+    (fp_text reference J5 (at 2.54 2.413 180) (layer F.SilkS)
+      (effects (font (size 0.762 0.762) (thickness 0.127)))
+    )
+    (fp_text value TC2030-CTX (at 0 -5) (layer F.Fab)
+      (effects (font (size 0.762 0.762) (thickness 0.127)))
+    )
+    (pad 1 smd circle (at -1.27 0.635) (size 0.7874 0.7874) (layers F.Cu F.Mask)
+      (net 1 +3V3))
+    (pad 2 smd circle (at -1.27 -0.635) (size 0.7874 0.7874) (layers F.Cu F.Mask)
+      (net 7 /SWDIO))
+    (pad 3 smd circle (at 0 0.635) (size 0.7874 0.7874) (layers F.Cu F.Mask)
+      (net 9 /nRST))
+    (pad 4 smd circle (at 0 -0.635) (size 0.7874 0.7874) (layers F.Cu F.Mask)
+      (net 8 /SWDCLK))
+    (pad 5 smd circle (at 1.27 0.635) (size 0.7874 0.7874) (layers F.Cu F.Mask)
+      (net 4 GNDD))
+    (pad 6 smd circle (at 1.27 -0.635) (size 0.7874 0.7874) (layers F.Cu F.Mask)
+      (net 32 "Net-(J5-Pad6)"))
+    (pad "" np_thru_hole circle (at 2.54 1.016) (size 0.9906 0.9906) (drill 0.9906) (layers *.Cu *.Mask))
+    (pad "" np_thru_hole circle (at 2.54 -1.016) (size 0.9906 0.9906) (drill 0.9906) (layers *.Cu *.Mask))
+    (pad "" np_thru_hole circle (at -2.54 0) (size 0.9906 0.9906) (drill 0.9906) (layers *.Cu *.Mask))
+  )
   (module alvarop:2450FM07A0029T (layer F.Cu)
     (at 181.9685 94.996)
@@
     )
   )
-  (module alvarop:TC2030-NL (layer F.Cu)
-    (at 187.198 99.441)
-    (fp_text reference J5 (at 2.54 2.413 180) (layer F.SilkS)
-      (effects (font (size 0.762 0.762) (thickness 0.127)))
-    )
-    (fp_text value TC2030-CTX (at 0 -5) (layer F.Fab)
-      (effects (font (size 0.762 0.762) (thickness 0.127)))
-    )
-    (pad 1 smd circle (at -1.27 0.635) (size 0.7874 0.7874) (layers F.Cu F.Paste F.Mask)
-      (net 1 +3V3))
-    (pad 2 smd circle (at -1.27 -0.635) (size 0.7874 0.7874) (layers F.Cu F.Paste F.Mask)
-      (net 7 /SWDIO))
-    (pad 3 smd circle (at 0 0.635) (size 0.7874 0.7874) (layers F.Cu F.Paste F.Mask)
-      (net 9 /nRST))
-    (pad 4 smd circle (at 0 -0.635) (size 0.7874 0.7874) (layers F.Cu F.Paste F.Mask)
-      (net 8 /SWDCLK))
-    (pad 5 smd circle (at 1.27 0.635) (size 0.7874 0.7874) (layers F.Cu F.Paste F.Mask)
-      (net 4 GNDD))
-    (pad 6 smd circle (at 1.27 -0.635) (size 0.7874 0.7874) (layers F.Cu F.Paste F.Mask)
-      (net 32 "Net-(J5-Pad6)"))
-    (pad "" np_thru_hole circle (at 2.54 1.016) (size 0.9906 0.9906) (drill 0.9906) (layers *.Cu *.Mask))
-    (pad "" np_thru_hole circle (at 2.54 -1.016) (size 0.9906 0.9906) (drill 0.9906) (layers *.Cu *.Mask))
-    (pad "" np_thru_hole circle (at -2.54 0) (size 0.9906 0.9906) (drill 0.9906) (layers *.Cu *.Mask))
-  )
   (module Resistors_SMD:R_0402 (layer F.Cu)
